Commit message: fixed a subtle bug in urdf interpretation of kdl_parser_py (#187)
* fix for unspecified origin RPY and added test for omitted rpy

File: kdl_parser_py/test/test.urdf (robot description, URDF)
Before this commit: robot physics, 11 links, 10 joints
Joints:
- joint left_gripper_joint: origin xyz=0.2 0.01 0 rpy=0 0 0 -> xyz=0.2 0.01 0
